File: Hardware/Controller/Controller.sch (KiCad schematic (older format))
At the start: 60 parts, among them J1 8P8C, J2 LCD Header, J3 USB_B_Micro, J4 S88 ShiftRegister, J5 Screw_Terminal_01x05, SW1 Rotary_Encoder_Switch, SW2 SW_Push_Dual, SW3 SW_Push_Dual, SW4 SW_Push_Dual, SW5 SW_Push_Dual, SW6 SW_Push_Dual, SW7 Shift, SW8 Stop, U1 ESP32-WROOM-32, U2 TJA1051T, U3 74LS367, U4 CH340C, U5 XM1584

Commit message: Switched to all-SMD Buttons
Parts:
- SW2: value SW_Push_Dual -> SW_F0; footprint Button_Switch_THT:SW_TH_Tactile_Omron_B3F-10xx -> Button_Switch_SMD:SW_SPST_B3S-1000; symbol Switch:SW_Push_Dual -> Switch:SW_Push
- SW3: value SW_Push_Dual -> SW_F1; footprint Button_Switch_THT:SW_TH_Tactile_Omron_B3F-10xx -> Button_Switch_SMD:SW_SPST_B3S-1000; symbol Switch:SW_Push_Dual -> Switch:SW_Push
- SW4: value SW_Push_Dual -> SW_F2; footprint Button_Switch_THT:SW_TH_Tactile_Omron_B3F-10xx -> Button_Switch_SMD:SW_SPST_B3S-1000; symbol Switch:SW_Push_Dual -> Switch:SW_Push
- SW5: value SW_Push_Dual -> SW_F3; footprint Button_Switch_THT:SW_TH_Tactile_Omron_B3F-10xx -> Button_Switch_SMD:SW_SPST_B3S-1000; symbol Switch:SW_Push_Dual -> Switch:SW_Push
- SW6: value SW_Push_Dual -> SW_F4; footprint Button_Switch_THT:SW_TH_Tactile_Omron_B3F-10xx -> Button_Switch_SMD:SW_SPST_B3S-1000; symbol Switch:SW_Push_Dual -> Switch:SW_Push
- SW7, SW8: footprint Button_Switch_THT:SW_TH_Tactile_Omron_B3F-10xx -> Button_Switch_SMD:SW_SPST_B3S-1000; symbol Switch:SW_Push_Dual -> Switch:SW_Push
Connections:
- net GND: no longer SW2.4, SW3.4, SW4.4, SW5.4, SW6.4, SW7.4, SW8.4
- net I2C_SCL: now also U1.12 (IO27); no longer U1.11 (IO26)
- net I2C_SDA: now also U1.11 (IO26); no longer U1.12 (IO27)
- net F2: now reaches C5.2, R10.2, U1.13 (IO14)
- net F0: now reaches C3.2, R6.2, U1.14 (IO12)
- net F1: now reaches C4.2, R8.2, U1.16 (IO13)
- net F3: now reaches C6.2, R12.2, U1.23 (IO15)
- net GPIO0: now reaches U1.25 (IO0), U4.13 (~DTR)
- net F4: now reaches C7.2, R14.2, U1.27 (IO16)
- net Shift: now reaches C8.2, R16.2, U1.28 (IO17)
- net EN: now reaches C11.1, U1.3 (EN), U4.14 (~RTS)
- net Encoder_A: now reaches C1.2, R2.2, U1.30 (IO18)
- net Stop: now reaches C9.2, R18.2, U1.31 (IO19)
- net EncoderB: now reaches C2.2, R4.2, U1.33 (IO21)
- net RX0: now reaches U1.34 (RXD0/IO3), U4.3 (RXD)
- net TX0: now reaches U1.35 (TXD0/IO1), U4.2 (TXD)
- net Encoder_Button: now reaches C10.2, R20.1, U1.36 (IO22)
- net at R5.1, R6.1, SW2.1: no longer SW2.3
- net at R7.1, R8.1, SW3.1: no longer SW3.3
- net at R10.1, R9.1, SW4.1: no longer SW4.3
- net at R11.1, R12.1, SW5.1: no longer SW5.3
- net at R13.1, R14.1, SW6.1: no longer SW6.3
- net at R15.1, R16.1, SW7.1: no longer SW7.3
- net at R17.1, R18.1, SW8.1: no longer SW8.3
Changed lines of the file:
@@
 Wire Wire Line
 	9850 5350 9850 5600
-Wire Wire Line
-	9850 5850 9850 6300
 $Comp
 L RF_Module:ESP32-WROOM-32 U1
@@
 $EndComp
 $Comp
-L Switch:SW_Push_Dual SW2
+L Switch:SW_Push SW2
 U 1 1 5C6944B8
 P 8350 1750
 F 0 "SW2" H 8350 2035 50  0000 C CNN
-F 1 "SW_Push_Dual" H 8350 1944 50  0000 C CNN
-F 2 "Button_Switch_THT:SW_TH_Tactile_Omron_B3F-10xx" H 8350 1950 50  0001 C CNN
+F 1 "SW_F0" H 8350 1944 50  0000 C CNN
+F 2 "Button_Switch_SMD:SW_SPST_B3S-1000" H 8350 1950 50  0001 C CNN
 F 3 "" H 8350 1950 50  0001 C CNN
 	1    8350 1750
@@
 $EndComp
 $Comp
-L Switch:SW_Push_Dual SW3
+L Switch:SW_Push SW3
 U 1 1 5C694536
 P 8350 2400
 F 0 "SW3" H 8350 2685 50  0000 C CNN
-F 1 "SW_Push_Dual" H 8350 2594 50  0000 C CNN
-F 2 "Button_Switch_THT:SW_TH_Tactile_Omron_B3F-10xx" H 8350 2600 50  0001 C CNN
+F 1 "SW_F1" H 8350 2594 50  0000 C CNN
+F 2 "Button_Switch_SMD:SW_SPST_B3S-1000" H 8350 2600 50  0001 C CNN
 F 3 "" H 8350 2600 50  0001 C CNN
 	1    8350 2400
@@
 $EndComp
 $Comp
-L Switch:SW_Push_Dual SW4
+L Switch:SW_Push SW4
 U 1 1 5C694574
 P 8350 3000
 F 0 "SW4" H 8350 3285 50  0000 C CNN
-F 1 "SW_Push_Dual" H 8350 3194 50  0000 C CNN
-F 2 "Button_Switch_THT:SW_TH_Tactile_Omron_B3F-10xx" H 8350 3200 50  0001 C CNN
+F 1 "SW_F2" H 8350 3194 50  0000 C CNN
+F 2 "Button_Switch_SMD:SW_SPST_B3S-1000" H 8350 3200 50  0001 C CNN
 F 3 "" H 8350 3200 50  0001 C CNN
 	1    8350 3000
@@
 $EndComp
 $Comp
-L Switch:SW_Push_Dual SW5
+L Switch:SW_Push SW5
 U 1 1 5C6945BA
 P 8350 3650
 F 0 "SW5" H 8350 3935 50  0000 C CNN
-F 1 "SW_Push_Dual" H 8350 3844 50  0000 C CNN
-F 2 "Button_Switch_THT:SW_TH_Tactile_Omron_B3F-10xx" H 8350 3850 50  0001 C CNN
+F 1 "SW_F3" H 8350 3844 50  0000 C CNN
+F 2 "Button_Switch_SMD:SW_SPST_B3S-1000" H 8350 3850 50  0001 C CNN
 F 3 "" H 8350 3850 50  0001 C CNN
 	1    8350 3650
@@
 $EndComp
 $Comp
-L Switch:SW_Push_Dual SW6
+L Switch:SW_Push SW6
 U 1 1 5C69460C
 P 8350 4300
 F 0 "SW6" H 8350 4585 50  0000 C CNN
-F 1 "SW_Push_Dual" H 8350 4494 50  0000 C CNN
-F 2 "Button_Switch_THT:SW_TH_Tactile_Omron_B3F-10xx" H 8350 4500 50  0001 C CNN
+F 1 "SW_F4" H 8350 4494 50  0000 C CNN
+F 2 "Button_Switch_SMD:SW_SPST_B3S-1000" H 8350 4500 50  0001 C CNN
 F 3 "" H 8350 4500 50  0001 C CNN
 	1    8350 4300
@@
 $EndComp
 $Comp
-L Switch:SW_Push_Dual SW7
+L Switch:SW_Push SW7
 U 1 1 5C694662
 P 8350 4950
 F 0 "SW7" H 8350 5235 50  0000 C CNN
 F 1 "Shift" H 8350 5144 50  0000 C CNN
-F 2 "Button_Switch_THT:SW_TH_Tactile_Omron_B3F-10xx" H 8350 5150 50  0001 C CNN
+F 2 "Button_Switch_SMD:SW_SPST_B3S-1000" H 8350 5150 50  0001 C CNN
 F 3 "" H 8350 5150 50  0001 C CNN
 	1    8350 4950
@@
 $EndComp
 $Comp
-L Switch:SW_Push_Dual SW8
+L Switch:SW_Push SW8
 U 1 1 5C6946AE
 P 8350 5650
 F 0 "SW8" H 8350 5935 50  0000 C CNN
 F 1 "Stop" H 8350 5844 50  0000 C CNN
-F 2 "Button_Switch_THT:SW_TH_Tactile_Omron_B3F-10xx" H 8350 5850 50  0001 C CNN
+F 2 "Button_Switch_SMD:SW_SPST_B3S-1000" H 8350 5850 50  0001 C CNN
 F 3 "" H 8350 5850 50  0001 C CNN
 	1    8350 5650
@@
 $EndComp
 Wire Wire Line
-	8550 1750 8550 1950
-Wire Wire Line
 	8550 6100 8600 6100
-Connection ~ 8550 1950
-Wire Wire Line
-	8550 1950 8550 2400
 Connection ~ 8550 2400
-Wire Wire Line
-	8550 2400 8550 2600
-Connection ~ 8550 2600
-Wire Wire Line
-	8550 2600 8550 3000
 Connection ~ 8550 3000
-Wire Wire Line
-	8550 3000 8550 3200
-Connection ~ 8550 3200
-Wire Wire Line
-	8550 3200 8550 3650
 Connection ~ 8550 3650
-Wire Wire Line
-	8550 3650 8550 3850
-Connection ~ 8550 3850
-Wire Wire Line
-	8550 3850 8550 4300
 Connection ~ 8550 4300
-Wire Wire Line
-	8550 4300 8550 4500
-Connection ~ 8550 4500
-Wire Wire Line
-	8550 4500 8550 4950
 Connection ~ 8550 4950
-Wire Wire Line
-	8550 4950 8550 5150
-Connection ~ 8550 5150
-Wire Wire Line
-	8550 5150 8550 5650
 Connection ~ 8550 5650
-Wire Wire Line
-	8550 5650 8550 5850
-Connection ~ 8550 5850
-Wire Wire Line
-	8550 5850 8550 6100
 Wire Wire Line
 	8550 1750 8650 1750
@@
 	7800 1950 8150 1950
 Connection ~ 7800 1950
-Connection ~ 8150 1950
 Wire Wire Line
 	8150 2600 7800 2600
-Connection ~ 8150 2600
 Connection ~ 7800 2600
 Wire Wire Line
@@
 Wire Wire Line
 	8150 3200 7800 3200
-Connection ~ 8150 3200
 Connection ~ 7800 3200
 Wire Wire Line
@@
 Wire Wire Line
 	8150 3850 7800 3850
-Connection ~ 8150 3850
 Connection ~ 7800 3850
 Wire Wire Line
@@
 Wire Wire Line
 	8150 5850 7800 5850
-Connection ~ 8150 5850
 Connection ~ 7800 5850
 Wire Wire Line
@@
 Wire Wire Line
 	8150 4500 7800 4500
-Connection ~ 8150 4500
 Connection ~ 7800 4500
 Wire Wire Line
@@
 Wire Wire Line
 	8150 5150 7800 5150
-Connection ~ 8150 5150
 Connection ~ 7800 5150
 Wire Wire Line
@@
 $EndComp
 Wire Wire Line
-	2350 3400 2400 3400
-Wire Wire Line
-	2400 3400 2400 4750
+	2400 3300 2400 4750
 Wire Wire Line
 	2400 4750 1500 4750
 Wire Wire Line
-	2350 3300 2450 3300
-Wire Wire Line
-	2450 3300 2450 4850
+	2450 3400 2450 4850
 Wire Wire Line
 	2450 4850 1500 4850
@@
 	650  1150 1050 1150
 Connection ~ 650  1150
+Wire Wire Line
+	8550 1750 8550 2400
+Wire Wire Line
+	8550 2400 8550 3000
+Wire Wire Line
+	8550 3000 8550 3650
+Wire Wire Line
+	8550 3650 8550 4300
+Wire Wire Line
+	8550 4300 8550 4950
+Wire Wire Line
+	8550 4950 8550 5650
+Wire Wire Line
+	8550 5650 8550 6100
+Wire Wire Line
+	9850 5850 9850 6300
+Wire Wire Line
+	2450 3400 2350 3400
+Wire Wire Line
+	2400 3300 2350 3300
+Text Label 6900 2250 0    50   ~ 0
+F0
+Text Label 6950 2850 0    50   ~ 0
+F1
+Text Label 6900 3450 0    50   ~ 0
+F2
+Text Label 6850 4050 0    50   ~ 0
+F3
+Text Label 6850 4700 0    50   ~ 0
+F4
+Text Label 6850 5400 0    50   ~ 0
+Shift
+Text Label 6850 6100 0    50   ~ 0
+Stop
+Text Label 6650 1050 0    50   ~ 0
+Encoder_A
+Text Label 6650 1650 0    50   ~ 0
+EncoderB
+Text Label 9500 1050 0    50   ~ 0
+Encoder_Button
+Text Label 2850 1600 0    50   ~ 0
+TX0
+Text Label 2850 1800 0    50   ~ 0
+RX0
+Text Label 2850 1500 0    50   ~ 0
+GPIO0
+Text Label 2850 700  0    50   ~ 0
+EN
 $EndSCHEMATC
