File: Hardware/ControllerTHT/ControllerTHT.kicad_pcb (KiCad board)
At the start: 2 copper layers, 40 x 107.5 mm, 59 parts, among them J1 8P8C, J2 LCD Header, J3 USB_B_Micro, J4 S88, J5 Screw_Terminal_01x05, SW1 Rotary_Encoder_Switch, SW2 SW_F0, SW3 SW_F1, SW4 SW_F2, SW5 SW_F3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

Commit message: More tinkering with Footprints
Parts:
- added U5: D24V10F3, Controller:D24V10F3, F.Cu at (78.7, 26.7)
- added U6: DOIT_ESP32_DEVKIT_V1, Controller:ESP32-DEVKITV1, F.Cu at (121.9, 119.4)
- C1, C10, C11, C2, C3, C4, C5, C6, C7, C8, C9: footprint Capacitor_SMD:C_0805_2012Metric_Pad1.15x1.40mm_HandSolder -> Capacitor_THT:C_Disc_D3.4mm_W2.1mm_P2.50mm
- C12: footprint Capacitor_SMD:CP_Elec_6.3x7.7 -> Capacitor_THT:CP_Radial_D10.0mm_P5.00mm
- C13: footprint Capacitor_Tantalum_SMD:CP_EIA-3216-18_Kemet-A_Pad1.58x1.35mm_HandSolder -> Capacitor_THT:CP_Radial_D5.0mm_P2.50mm
- D1, D2: footprint Diode_SMD:D_0603_1608Metric_Pad1.05x0.95mm_HandSolder -> Diode_THT:D_A-405_P7.62mm_Horizontal
- R1, R10, R11, R12, R13, R14, R15, R16, R17, R18, R19, R2, R20, R3, R4, R5, R6, R7, R8, R9: footprint Resistor_SMD:R_0603_1608Metric_Pad1.05x0.95mm_HandSolder -> Resistor_THT:R_Axial_DIN0207_L6.3mm_D2.5mm_P10.16mm_Horizontal
- SW2, SW3, SW4, SW5, SW6, SW7, SW8: footprint Button_Switch_SMD:SW_SPST_B3S-1000 -> Button_Switch_THT:SW_PUSH_6mm_H9.5mm
- U3: footprint Package_SO:SOP-16_4.4x10.4mm_P1.27mm -> Package_DIP:DIP-16_W7.62mm_Socket
- moved SW2 117.9 mm to (19.1, 63.5)
- moved SW1 115.0 mm to (213.4, 48.3), turned to 180 degrees
- moved SW4 114.0 mm to (44.5, 63.5)
- moved SW6 113.7 mm to (34.3, 74.9)
- moved SW5 113.5 mm to (24.1, 74.9)
- moved J3 109.0 mm to (61.8, 105.5)
- moved R2 104.5 mm to (221.0, 48.3), turned to 90 degrees
- moved SW8 99.3 mm to (47.0, 54.6), turned to 90 degrees
- moved R1 95.9 mm to (215.9, 48.3), turned to 270 degrees
- moved C1 89.5 mm to (223.5, 35.6), turned to 270 degrees
- moved J2 82.9 mm to (31.2, 40.6), turned to 90 degrees
- moved C10 82.7 mm to (200.7, 35.6), turned to 90 degrees
- moved U4 80.5 mm to (49.6, 87.0)
- moved C2 77.9 mm to (213.4, 35.6), turned to 90 degrees
- moved U1 68.2 mm to (129.5, 119.4), turned to 270 degrees
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Connections:
- U1 pad 10: (no net) -> /IO25
- U1 pad 24: (no net) -> /IO2
- U1 pad 37: (no net) -> /IO23
- U1 pad 4: (no net) -> /VP
- U1 pad 5: (no net) -> /VN
Routing:
- net GND: track 0.00 -> 59.2 mm, vias 0 -> 4
- net VCC: track 0.00 -> 40.6 mm, vias 0 -> 2
- net /F2: track 0.00 -> 14.7 mm
- net /F1: track 0.00 -> 14.7 mm
- net /IO2: track 0.00 -> 11.7 mm
- net /F0: track 0.00 -> 11.5 mm
- net /CANRx: track 0.00 -> 11.0 mm
- net /F3: track 0.00 -> 11.0 mm
- net Net-(R3-Pad1): track 0.00 -> 10.2 mm
- net /EncoderB: track 0.00 -> 10.1 mm
- net /Encoder_Button: track 0.00 -> 10.1 mm
- net /Shift: track 0.00 -> 9.69 mm
- net /I2C_SDA: track 0.00 -> 9.69 mm
- net /F4: track 0.00 -> 8.42 mm
- net /I2C_SCL: track 0.00 -> 8.42 mm
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
Commit message: Intermediate steps
Parts:
- added C14: 10u, Capacitor_THT:CP_Radial_D10.0mm_P5.00mm, F.Cu at (40.5, 67.5)
- added C15: 100n, Capacitor_THT:C_Disc_D3.4mm_W2.1mm_P2.50mm, F.Cu at (25.2, 80.2)
- added J6: Conn_01x05_Female, Connector_PinHeader_2.54mm:PinHeader_1x05_P2.54mm_Vertical, F.Cu at (22.9, 24.1)
- added J7: Conn_01x02_Female, Connector_PinHeader_2.54mm:PinHeader_1x02_P2.54mm_Vertical, F.Cu at (26.7, 26.7)
- added J8: Conn_01x02_Female, Connector_PinHeader_2.54mm:PinHeader_1x02_P2.54mm_Vertical, F.Cu at (35.6, 24.1)
- added Q1: BC547, Package_TO_SOT_THT:TO-92_Inline, F.Cu at (50.7, 65.0)
- added Q2: BC547, Package_TO_SOT_THT:TO-92_Inline, F.Cu at (46.7, 76.5)
- added R21: 10k, Resistor_THT:R_Axial_DIN0207_L6.3mm_D2.5mm_P10.16mm_Horizontal, F.Cu at (25.2, 63.8)
- added R22: 10k, Resistor_THT:R_Axial_DIN0207_L6.3mm_D2.5mm_P10.16mm_Horizontal, F.Cu at (25.2, 67.8)
- added SW10: SW_Push, Button_Switch_THT:SW_PUSH_6mm, F.Cu at (36.2, 75.3)
- added SW9: SW_Push, Button_Switch_THT:SW_PUSH_6mm, F.Cu at (25.7, 71.9)
- U5: moved to B.Cu
- moved U1 119.7 mm to (50.8, 29.2)
- moved U6 119.7 mm to (43.2, 29.2)
- moved C10 116.5 mm to (255.3, 138.4)
- moved C2 116.5 mm to (268.0, 138.4)
- moved R19 116.5 mm to (247.7, 156.2)
- moved R4 116.5 mm to (273.1, 146.1)
- moved SW1 116.5 mm to (268.0, 151.1)
- moved C1 116.5 mm to (278.1, 138.4)
- moved R1 116.5 mm to (270.5, 151.1)
- moved R2 116.5 mm to (275.6, 151.1)
- moved R3 116.5 mm to (278.1, 146.1)
- moved R20 116.5 mm to (250.2, 135.9)
- moved C5 88.8 mm to (243.0, 86.3)
- moved R10 88.8 mm to (234.9, 99.9)
- moved R14 88.8 mm to (220.4, 115.1)
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Connections:
- J3 pad 4: (no net) -> Net-(J3-Pad4)
- U4 pad 13: /GPIO0 -> Net-(Q2-Pad3)
- U4 pad 14: /EN -> Net-(Q1-Pad3)
Routing:
- net /USB-: track 0.00 -> 15.1 mm
- net /USB+: track 0.00 -> 14.5 mm
- net /VinUsb: track 0.00 -> 6.47 mm
- net GND: track 59.2 -> 64.7 mm
- net Net-(J3-Pad4): track 0.00 -> 4.40 mm
- net /BOARD_TX0: track 4.46 -> 7.88 mm
- net /BOARD_RX0: track 4.46 -> 7.36 mm
Other:
- board outline removed

Commit message: Updated all boards
ESP32Breakout now with S88 driver.
ESP32Breakout has the auto-reset circut removed.
Parts:
- removed SW10: SW_Push, Button_Switch_THT:SW_PUSH_6mm
Connections:
- C8 pad 2: /Shift -> /GPIO0
- R16 pad 2: /Shift -> /GPIO0
- U1 pad 27: /Shift -> (no net)
- U6 pad 6: /Shift -> /GPIO0
Routing:
- net /Shift: track 9.69 -> 0.00 mm
- net /GPIO0: track 0.00 -> 8.44 mm
