File: Hardware/ControllerTHT/ControllerTHT.sch (KiCad schematic (older format))
At the start: 60 parts, among them J1 8P8C, J2 LCD Header, J3 USB_B_Micro, J4 S88, J5 Screw_Terminal_01x05, SW1 Rotary_Encoder_Switch, SW2 SW_F0, SW3 SW_F1, SW4 SW_F2, SW5 SW_F3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

Commit message: More tinkering with Footprints
Parts:
- removed U5: XM1584, Controller:XM1584, symbol ControllerParts:XM1584
- added U5: D24V10F3, Controller:D24V10F3, symbol ControllerParts:D24V10F3
- added U6: DOIT_ESP32_DEVKIT_V1, Controller:ESP32-DEVKITV1, symbol ControllerParts:DOIT_ESP32_DEVKIT_V1
- C1, C10, C11, C2, C3, C4, C5, C6, C7, C8, C9: footprint Capacitor_SMD:C_0805_2012Metric_Pad1.15x1.40mm_HandSolder -> Capacitor_THT:C_Disc_D3.4mm_W2.1mm_P2.50mm
- C12: footprint Capacitor_SMD:CP_Elec_6.3x7.7 -> Capacitor_THT:CP_Radial_D10.0mm_P5.00mm
- C13: footprint Capacitor_Tantalum_SMD:CP_EIA-3216-18_Kemet-A_Pad1.58x1.35mm_HandSolder -> Capacitor_THT:CP_Radial_D5.0mm_P2.50mm
- D1, D2: footprint Diode_SMD:D_0603_1608Metric_Pad1.05x0.95mm_HandSolder -> Diode_THT:D_A-405_P7.62mm_Horizontal
- R1, R10, R11, R12, R13, R14, R15, R16, R17, R18, R19, R2, R20, R3, R4, R5, R6, R7, R8, R9: footprint Resistor_SMD:R_0603_1608Metric_Pad1.05x0.95mm_HandSolder -> Resistor_THT:R_Axial_DIN0207_L6.3mm_D2.5mm_P10.16mm_Horizontal
- SW2, SW3, SW4, SW5, SW6, SW7, SW8: footprint Button_Switch_SMD:SW_SPST_B3S-1000 -> Button_Switch_THT:SW_PUSH_6mm_H9.5mm
- U3: footprint Package_SO:SOP-16_4.4x10.4mm_P1.27mm -> Package_DIP:DIP-16_W7.62mm_Socket
Connections:
- net labels added: IO2, IO23, IO25, VN, VP
- net labels removed: VinTerminal
- wire segments 280 -> 254
- no-connect marks 1 -> 24
Other:
- moved on the sheet: C11

Commit message: Intermediate steps
Parts:
- added C14: 10u, Capacitor_THT:CP_Radial_D10.0mm_P5.00mm, symbol Device:CP
- added C15: 100n, Capacitor_THT:C_Disc_D3.4mm_W2.1mm_P2.50mm, symbol Device:C
- added J6: Conn_01x05_Female, Connector_PinHeader_2.54mm:PinHeader_1x05_P2.54mm_Vertical, symbol Connector:Conn_01x05_Female
- added J7, J8: Conn_01x02_Female, Connector_PinHeader_2.54mm:PinHeader_1x02_P2.54mm_Vertical, symbol Connector:Conn_01x02_Female
- added Q1, Q2: BC547, Package_TO_SOT_THT:TO-92_Inline, symbol Transistor_BJT:BC547
- added R21, R22: 10k, Resistor_THT:R_Axial_DIN0207_L6.3mm_D2.5mm_P10.16mm_Horizontal, symbol Device:R
- added SW10, SW9: SW_Push, Button_Switch_THT:SW_PUSH_6mm, symbol Switch:SW_Push
Connections:
- wire segments 254 -> 287
- no-connect marks 24 -> 23
Other:
- moved on the sheet: C11, U1

Commit message: Updated all boards
ESP32Breakout now with S88 driver.
ESP32Breakout has the auto-reset circut removed.
Parts:
- removed SW10: SW_Push, Button_Switch_THT:SW_PUSH_6mm, symbol Switch:SW_Push
Connections:
- wire segments 287 -> 284
Changed lines of the file:
@@
 Text Label 6850 4700 0    50   ~ 0
 F4
-Text Label 6850 5400 0    50   ~ 0
+Text Label 6950 5400 0    50   ~ 0
 Shift
 Text Label 6850 6100 0    50   ~ 0
@@
 Wire Wire Line
 	3800 2750 2800 2750
-Wire Wire Line
-	2800 2450 3350 2450
 Text Label 5650 1150 0    50   ~ 0
 S88_CLOCK
@@
 Text Label 3150 2550 0    50   ~ 0
 F4
-Text Label 3150 2450 0    50   ~ 0
-Shift
 Text Label 3150 2750 0    50   ~ 0
 Encoder_A
@@
 	0    1    1    0
 $EndComp
-$Comp
-L Switch:SW_Push SW10
-U 1 1 5D10FE38
-P 3650 4300
-F 0 "SW10" H 3650 4585 50  0000 C CNN
-F 1 "SW_Push" H 3650 4494 50  0000 C CNN
-F 2 "Button_Switch_THT:SW_PUSH_6mm" H 3650 4500 50  0001 C CNN
-F 3 "~" H 3650 4500 50  0001 C CNN
-	1    3650 4300
-	1    0    0    -1
-$EndComp
 Wire Wire Line
 	1350 2500 1000 2500
@@
 Wire Wire Line
 	3450 4500 3550 4500
-Connection ~ 3450 4300
-Wire Wire Line
-	3850 4300 4100 4300
-Wire Wire Line
-	4100 4300 4100 4500
 Wire Wire Line
 	3850 4500 4100 4500
-Connection ~ 4100 4500
 Wire Wire Line
 	4100 4500 4100 4600
@@
 	1    0    0    -1
 $EndComp
+Text Label 6700 5400 0    50   ~ 0
+GPIO0
 $EndSCHEMATC
