File: Hardware/ESP32Breakout/ESP32Breakout.sch (KiCad schematic (older format))
At the start: 36 parts, among them J1 8P8C, J10 ESP32 BO L, J11 RJ45 BO, J12 CAN BO, J2 LCD Header, J3 USB_B_Micro, J4 Conn_01x02_Male, J5 Screw_Terminal_01x05, J6 USBConn BO, J7 USB BO L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

Commit message: Fixup of holes and labels
Parts:
- H3, H4, H5, H6: footprint MountingHole:MountingHole_2.5mm_Pad_Via -> MountingHole:MountingHole_3.2mm_M3_Pad_Via
Changed lines of the file:
@@
 EESchema Schematic File Version 4
+LIBS:ESP32Breakout-cache
 EELAYER 29 0
 EELAYER END
@@
 F 0 "H6" H 10750 5796 50  0000 L CNN
 F 1 "PCB Screw" H 10750 5705 50  0000 L CNN
-F 2 "MountingHole:MountingHole_2.5mm_Pad_Via" H 10650 5750 50  0001 C CNN
+F 2 "MountingHole:MountingHole_3.2mm_M3_Pad_Via" H 10650 5750 50  0001 C CNN
 F 3 "~" H 10650 5750 50  0001 C CNN
 	1    10650 5750
@@
 F 0 "H5" H 10750 5546 50  0000 L CNN
 F 1 "PCB Screw" H 10750 5455 50  0000 L CNN
-F 2 "MountingHole:MountingHole_2.5mm_Pad_Via" H 10650 5500 50  0001 C CNN
+F 2 "MountingHole:MountingHole_3.2mm_M3_Pad_Via" H 10650 5500 50  0001 C CNN
 F 3 "~" H 10650 5500 50  0001 C CNN
 	1    10650 5500
@@
 F 0 "H4" H 10750 5296 50  0000 L CNN
 F 1 "PCB Screw" H 10750 5205 50  0000 L CNN
-F 2 "MountingHole:MountingHole_2.5mm_Pad_Via" H 10650 5250 50  0001 C CNN
+F 2 "MountingHole:MountingHole_3.2mm_M3_Pad_Via" H 10650 5250 50  0001 C CNN
 F 3 "~" H 10650 5250 50  0001 C CNN
 	1    10650 5250
@@
 F 0 "H3" H 10750 5046 50  0000 L CNN
 F 1 "PCB Screw" H 10750 4955 50  0000 L CNN
-F 2 "MountingHole:MountingHole_2.5mm_Pad_Via" H 10650 5000 50  0001 C CNN
+F 2 "MountingHole:MountingHole_3.2mm_M3_Pad_Via" H 10650 5000 50  0001 C CNN
 F 3 "~" H 10650 5000 50  0001 C CNN
 	1    10650 5000

Commit message: Updated all boards
ESP32Breakout now with S88 driver.
ESP32Breakout has the auto-reset circut removed.
Parts:
- removed C14: 10u, Capacitor_THT:CP_Radial_D10.0mm_P5.00mm, symbol Device:CP
- removed J7: USB BO L, Connector_PinHeader_2.54mm:PinHeader_1x08_P2.54mm_Vertical, symbol Connector:Conn_01x08_Female
- removed J9: USB BO R, Connector_PinHeader_2.54mm:PinHeader_1x08_P2.54mm_Vertical, symbol Connector:Conn_01x08_Female
- removed Q1, Q2: BC547, Package_TO_SOT_THT:TO-92_Inline, symbol Transistor_BJT:BC547
- removed R21, R22: 10k, Resistor_THT:R_Axial_DIN0207_L6.3mm_D2.5mm_P10.16mm_Horizontal, symbol Device:R
- removed U2: TJA1051T, Package_SO:SOIC-8_3.9x4.9mm_P1.27mm, symbol Interface_CAN_LIN:TJA1051T
- removed U4: CH340C, Package_SO:SOIC-16_3.9x9.9mm_P1.27mm, symbol Interface_USB:CH340G
- added J13: Conn_01x02_Male, Connector_PinHeader_2.54mm:PinHeader_1x02_P2.54mm_Vertical, symbol Connector:Conn_01x02_Male
- added J7: S88 Header, Connector_PinHeader_2.54mm:PinHeader_1x06_P2.54mm_Vertical, symbol Connector:Conn_01x06_Male
- added J9: 8P8C, Connector_RJ:RJ45_Amphenol_54602-x08_Horizontal, symbol Connector:8P8C
- added U2: SN65HVD230, Package_SO:SOIC-8_3.9x4.9mm_P1.27mm, symbol Interface_CAN_LIN:SN65HVD230
- added U4: 74LS367, Package_SO:SOP-16_4.55x10.3mm_P1.27mm, symbol 74xx:74LS367
- added U6: CH340G, Package_SO:SOIC-16_3.9x9.9mm_P1.27mm, symbol Interface_USB:CH340G
- J2: footprint Connector_PinHeader_2.54mm:PinHeader_1x04_P2.54mm_Vertical -> Connector_PinHeader_2.54mm:PinHeader_1x06_P2.54mm_Vertical; symbol Connector:Conn_01x04_Female -> Connector:Conn_01x06_Male
Connections:
- net labels added: GPIO0-SER, IO12, IO13, IO14, IO15, IO16, IO17, IO19, IO33, IO34, S88_CLOCK, S88_PS, S88_RESET
- net labels removed: !DTR, !RTS, Encoder_Button, F0, F1, F2, F3, F4, IO23, Shift, Stop
- wire segments 229 -> 240
- no-connect marks 10 -> 11
Other:
- moved on the sheet: J11, J12, J4, SW9, U3
