File: Hardware/S88Driver/S88Driver.kicad_pcb (KiCad board)
At the start: 2 copper layers, 28 x 40 mm, 8 parts, among them J1 Conn_01x06_Male, J2 Conn_01x06_Female, U1 74LS367

Commit message: Updates projects for manufacturing
Other:
- outline, holes or cut-outs redrawn
- board text added: "RR32Can S88 Buffer v1.0"
- board text added: "To Bus"
- board text added: "To uC"
- board text added: "VCC RES LD CLK GND DATA"
Changed lines of the file:
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@@
   (general
     (thickness 1.6)
-    (drawings 5)
+    (drawings 13)
     (tracks 35)
     (zones 0)
@@
   )
   (setup
-    (last_trace_width 1)
+    (last_trace_width 0.25)
     (user_trace_width 1)
     (trace_clearance 0.2)
@@
     (pad_to_mask_clearance 0.051)
     (solder_mask_min_width 0.25)
-    (aux_axis_origin 0 0)
-    (visible_elements FFFFFF7F)
+    (aux_axis_origin 20 20)
+    (visible_elements 7FFFFFFF)
     (pcbplotparams
-      (layerselection 0x010fc_ffffffff)
-      (usegerberextensions false)
+      (layerselection 0x010f0_ffffffff)
+      (usegerberextensions true)
       (usegerberattributes false)
       (usegerberadvancedattributes false)
@@
       (viasonmask false)
       (mode 1)
-      (useauxorigin false)
+      (useauxorigin true)
       (hpglpennumber 1)
       (hpglpenspeed 20)
@@
       (outputformat 1)
       (mirror false)
-      (drillshape 1)
+      (drillshape 0)
       (scaleselection 1)
-      (outputdirectory ""))
+      (outputdirectory "gerber"))
   )
   (net 0 "")
@@
     (add_net "Net-(J2-Pad4)")
     (add_net "Net-(J2-Pad5)")
-    (add_net "Net-(U1-Pad11)")
-    (add_net "Net-(U1-Pad13)")
-    (add_net "Net-(U1-Pad9)")
     (add_net VCC)
   )
@@
     (tags "mounting hole 2.7mm")
     (attr virtual)
-    (fp_text reference H4 (at 0 -3.7) (layer F.SilkS)
+    (fp_text reference H4 (at 0 -3.7) (layer F.SilkS) hide
       (effects (font (size 1 1) (thickness 0.15)))
     )
@@
     (tags "mounting hole 2.7mm")
     (attr virtual)
-    (fp_text reference H3 (at 0 -3.7) (layer F.SilkS)
+    (fp_text reference H3 (at 0 -3.7) (layer F.SilkS) hide
       (effects (font (size 1 1) (thickness 0.15)))
     )
@@
     (tags "mounting hole 2.7mm")
     (attr virtual)
-    (fp_text reference H2 (at 0 -3.7) (layer F.SilkS)
+    (fp_text reference H2 (at 0 -3.7) (layer F.SilkS) hide
       (effects (font (size 1 1) (thickness 0.15)))
     )
@@
     (tags "mounting hole 2.7mm")
     (attr virtual)
-    (fp_text reference H1 (at 0 -3.7) (layer F.SilkS)
+    (fp_text reference H1 (at 0 -3.7) (layer F.SilkS) hide
       (effects (font (size 1 1) (thickness 0.15)))
     )
@@
     (descr "Through hole angled socket strip, 1x06, 2.54mm pitch, 8.51mm socket length, single row (from Kicad 4.0.7), script generated")
     (tags "Through hole angled socket strip THT 1x06 2.54mm single row")
-    (fp_text reference J2 (at -4.38 -2.77 90) (layer F.SilkS)
+    (fp_text reference J2 (at -3 -2.77 90) (layer F.SilkS)
       (effects (font (size 1 1) (thickness 0.15)))
     )
@@
     )
   )
-  (target plus (at 20 20) (size 5) (width 0.05) (layer Edge.Cuts))
-  (gr_line (start 48 20) (end 48 60) (layer Edge.Cuts) (width 0.1))
-  (gr_line (start 20 20) (end 48 20) (layer Edge.Cuts) (width 0.1))
-  (gr_line (start 20 60) (end 20 20) (layer Edge.Cuts) (width 0.1))
-  (gr_line (start 48 60) (end 20 60) (layer Edge.Cuts) (width 0.1))
+  (gr_text "RR32Can\nS88 Buffer v1.0" (at 46 48 90) (layer F.SilkS)
+    (effects (font (size 1 1) (thickness 0.15)))
+  )
+  (gr_text "To uC" (at 34 48) (layer F.SilkS)
+    (effects (font (size 1 1) (thickness 0.15)))
+  )
+  (gr_text "VCC\nRES\nLD\nCLK\nGND\nDATA" (at 34 53 90) (layer F.SilkS)
+    (effects (font (size 1 1) (thickness 0.15)) (justify right))
+  )
+  (gr_text "VCC\nRES\nLD\nCLK\nGND\nDATA" (at 34 32 90) (layer F.SilkS)
+    (effects (font (size 1 1) (thickness 0.15)) (justify right))
+  )
+  (gr_text "To Bus" (at 45 29) (layer F.SilkS)
+    (effects (font (size 1 1) (thickness 0.15)))
+  )
+  (gr_arc (start 23 57) (end 20 57) (angle -90) (layer Edge.Cuts) (width 0.1))
+  (gr_arc (start 45 57) (end 45 60) (angle -90) (layer Edge.Cuts) (width 0.1))
+  (gr_arc (start 45 23) (end 48 23) (angle -90) (layer Edge.Cuts) (width 0.1))
+  (gr_arc (start 23 23) (end 23 20) (angle -90) (layer Edge.Cuts) (width 0.1))
+  (gr_line (start 48 23) (end 48 57) (layer Edge.Cuts) (width 0.1))
+  (gr_line (start 23 20) (end 45 20) (layer Edge.Cuts) (width 0.1))
+  (gr_line (start 20 57) (end 20 23) (layer Edge.Cuts) (width 0.1))
+  (gr_line (start 45 60) (end 23 60) (layer Edge.Cuts) (width 0.1))
   (via (at 36 40) (size 0.8) (drill 0.4) (layers F.Cu B.Cu) (net 1))
   (segment (start 26 30) (end 22 34) (width 1) (layer F.Cu) (net 2))

Commit message: Further updates
Parts:
- added J3: Conn_01x06_Male, Connector_PinSocket_2.54mm:PinSocket_1x06_P2.54mm_Vertical, F.Cu at (40.0, 21.6)
Routing:
- net VCC: track 47.3 -> 55.7 mm
- net Net-(J2-Pad5): track 8.28 -> 16.7 mm
- net Net-(J2-Pad4): track 7.22 -> 15.6 mm
- net Net-(J2-Pad3): track 7.83 -> 16.2 mm
- net /S88_DATA: track 27.3 -> 34.6 mm
Changed lines of the file:
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@@
     (thickness 1.6)
     (drawings 13)
-    (tracks 35)
+    (tracks 39)
     (zones 0)
-    (modules 8)
+    (modules 9)
     (nets 10)
   )
@@
   )
   (setup
-    (last_trace_width 0.25)
+    (last_trace_width 1)
     (user_trace_width 1)
     (trace_clearance 0.2)
@@
     (add_net "Net-(J2-Pad4)")
     (add_net "Net-(J2-Pad5)")
+    (add_net "Net-(U1-Pad11)")
+    (add_net "Net-(U1-Pad13)")
+    (add_net "Net-(U1-Pad9)")
     (add_net VCC)
+  )
+  (module Connector_PinSocket_2.54mm:PinSocket_1x06_P2.54mm_Vertical (layer F.Cu)
+    (at 40 21.59 270)
+    (descr "Through hole straight socket strip, 1x06, 2.54mm pitch, single row (from Kicad 4.0.7), script generated")
+    (tags "Through hole socket strip THT 1x06 2.54mm single row")
+    (fp_text reference J3 (at 0 -2.77 90) (layer F.SilkS)
+      (effects (font (size 1 1) (thickness 0.15)))
+    )
+    (fp_text value Conn_01x06_Male (at 0 15.47 90) (layer F.Fab)
+      (effects (font (size 1 1) (thickness 0.15)))
+    )
+    (fp_text user %R (at 0 6.35) (layer F.Fab)
+      (effects (font (size 1 1) (thickness 0.15)))
+    )
+    (fp_line (start -1.8 14.45) (end -1.8 -1.8) (layer F.CrtYd) (width 0.05))
+    (fp_line (start 1.75 14.45) (end -1.8 14.45) (layer F.CrtYd) (width 0.05))
+    (fp_line (start 1.75 -1.8) (end 1.75 14.45) (layer F.CrtYd) (width 0.05))
+    (fp_line (start -1.8 -1.8) (end 1.75 -1.8) (layer F.CrtYd) (width 0.05))
+    (fp_line (start 0 -1.33) (end 1.33 -1.33) (layer F.SilkS) (width 0.12))
+    (fp_line (start 1.33 -1.33) (end 1.33 0) (layer F.SilkS) (width 0.12))
+    (fp_line (start 1.33 1.27) (end 1.33 14.03) (layer F.SilkS) (width 0.12))
+    (fp_line (start -1.33 14.03) (end 1.33 14.03) (layer F.SilkS) (width 0.12))
+    (fp_line (start -1.33 1.27) (end -1.33 14.03) (layer F.SilkS) (width 0.12))
+    (fp_line (start -1.33 1.27) (end 1.33 1.27) (layer F.SilkS) (width 0.12))
+    (fp_line (start -1.27 13.97) (end -1.27 -1.27) (layer F.Fab) (width 0.1))
+    (fp_line (start 1.27 13.97) (end -1.27 13.97) (layer F.Fab) (width 0.1))
+    (fp_line (start 1.27 -0.635) (end 1.27 13.97) (layer F.Fab) (width 0.1))
+    (fp_line (start 0.635 -1.27) (end 1.27 -0.635) (layer F.Fab) (width 0.1))
+    (fp_line (start -1.27 -1.27) (end 0.635 -1.27) (layer F.Fab) (width 0.1))
+    (pad 6 thru_hole oval (at 0 12.7 270) (size 1.7 1.7) (drill 1) (layers *.Cu *.Mask)
+      (net 2 VCC))
+    (pad 5 thru_hole oval (at 0 10.16 270) (size 1.7 1.7) (drill 1) (layers *.Cu *.Mask)
+      (net 7 "Net-(J2-Pad5)"))
+    (pad 4 thru_hole oval (at 0 7.62 270) (size 1.7 1.7) (drill 1) (layers *.Cu *.Mask)
+      (net 8 "Net-(J2-Pad4)"))
+    (pad 3 thru_hole oval (at 0 5.08 270) (size 1.7 1.7) (drill 1) (layers *.Cu *.Mask)
+      (net 9 "Net-(J2-Pad3)"))
+    (pad 2 thru_hole oval (at 0 2.54 270) (size 1.7 1.7) (drill 1) (layers *.Cu *.Mask)
+      (net 1 GND))
+    (pad 1 thru_hole rect (at 0 0 270) (size 1.7 1.7) (drill 1) (layers *.Cu *.Mask)
+      (net 6 /S88_DATA))
+    (model ${KISYS3DMOD}/Connector_PinSocket_2.54mm.3dshapes/PinSocket_1x06_P2.54mm_Vertical.wrl
+      (at (xyz 0 0 0))
+      (scale (xyz 1 1 1))
+      (rotate (xyz 0 0 0))
+    )
   )
   (module MountingHole:MountingHole_2.7mm_M2.5_Pad_Via (layer F.Cu)
@@
   (segment (start 27.3 51) (end 28.850001 49.449999) (width 1) (layer B.Cu) (net 2))
   (segment (start 42 44.62) (end 39.46 44.62) (width 1) (layer B.Cu) (net 2))
+  (segment (start 27.3 30) (end 27.3 21.59) (width 1) (layer F.Cu) (net 2))
   (segment (start 29.84 51) (end 29.84 46.071004) (width 0.25) (layer F.Cu) (net 3))
   (segment (start 30.42501 45.485994) (end 30.42501 41.42501) (width 0.25) (layer F.Cu) (net 3))
@@
   (segment (start 39.46 39.54) (end 39.46 37) (width 0.25) (layer F.Cu) (net 5))
   (segment (start 35.50501 43.49499) (end 39.46 39.54) (width 0.25) (layer F.Cu) (net 5))
-  (segment (start 41.85 30) (end 45 33.15) (width 1) (layer F.Cu) (net 6))
-  (segment (start 40 30) (end 41.85 30) (width 1) (layer F.Cu) (net 6))
+  (segment (start 40 30) (end 40 21.59) (width 1) (layer F.Cu) (net 6))
+  (segment (start 41.85 51) (end 40 51) (width 1) (layer F.Cu) (net 6))
   (segment (start 45 47.85) (end 41.85 51) (width 1) (layer F.Cu) (net 6))
-  (segment (start 41.85 51) (end 40 51) (width 1) (layer F.Cu) (net 6))
-  (segment (start 45 33.15) (end 45 47.85) (width 1) (layer F.Cu) (net 6))
+  (segment (start 40 30) (end 45 35) (width 1) (layer F.Cu) (net 6))
+  (segment (start 45 35) (end 45 47.85) (width 1) (layer F.Cu) (net 6))
   (segment (start 29.84 33.92) (end 26.76 37) (width 1) (layer F.Cu) (net 7))
   (segment (start 29.84 30) (end 29.84 33.92) (width 1) (layer F.Cu) (net 7))
+  (segment (start 29.84 30) (end 29.84 21.59) (width 1) (layer F.Cu) (net 7))
   (segment (start 32.38 36.46) (end 31.84 37) (width 1) (layer F.Cu) (net 8))
   (segment (start 32.38 30) (end 32.38 36.46) (width 1) (layer F.Cu) (net 8))
+  (segment (start 32.38 30) (end 32.38 21.59) (width 1) (layer F.Cu) (net 8))
   (segment (start 34.92 35) (end 36.92 37) (width 1) (layer F.Cu) (net 9))
   (segment (start 34.92 30) (end 34.92 35) (width 1) (layer F.Cu) (net 9))
+  (segment (start 34.92 30) (end 34.92 21.59) (width 1) (layer F.Cu) (net 9))
   (zone (net 1) (net_name GND) (layer F.Cu) (hatch edge 0.508)
     (connect_pads (clearance 0.508))
