File: Hardware/SwitchboardConnector/SwitchboardConnector.kicad_pcb (KiCad board)
At the start: 2 copper layers, 5.1 x 25.4 mm, 1 part, among them J1 Conn_02x06_Odd_Even

Commit message: Further updates
Parts:
- added J2: Conn_01x06_Female, Connector_PinSocket_2.54mm:PinSocket_1x06_P2.54mm_Vertical, F.Cu at (29.2, 20.3)
Routing:
- net Net-(J1-Pad7): track 2.54 -> 5.08 mm
- net Net-(J1-Pad5): track 2.54 -> 5.08 mm
- net Net-(J1-Pad3): track 2.54 -> 5.08 mm
- net Net-(J1-Pad11): track 2.54 -> 5.08 mm
- net Net-(J1-Pad10): track 2.54 -> 5.08 mm
- net Net-(J1-Pad1): track 2.54 -> 5.08 mm
Other:
- board size 5.1 x 25.4 mm -> 7.6 x 25.4 mm
Changed lines of the file:
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@@
   (general
     (thickness 1.6)
-    (drawings 4)
-    (tracks 6)
+    (drawings 8)
+    (tracks 12)
     (zones 0)
-    (modules 1)
+    (modules 2)
     (nets 7)
   )
@@
     (solder_mask_min_width 0.25)
     (aux_axis_origin 22.86 13.97)
-    (visible_elements FFFFFF7F)
+    (visible_elements 7FFFFFFF)
     (pcbplotparams
       (layerselection 0x010f0_ffffffff)
@@
     (add_net "Net-(J1-Pad5)")
     (add_net "Net-(J1-Pad7)")
+  )
+  (module Connector_PinSocket_2.54mm:PinSocket_1x06_P2.54mm_Vertical (layer F.Cu)
+    (at 29.21 20.32)
+    (descr "Through hole straight socket strip, 1x06, 2.54mm pitch, single row (from Kicad 4.0.7), script generated")
+    (tags "Through hole socket strip THT 1x06 2.54mm single row")
+    (fp_text reference J2 (at 0 -2.77) (layer F.SilkS)
+      (effects (font (size 1 1) (thickness 0.15)))
+    )
+    (fp_text value Conn_01x06_Female (at 0 15.47) (layer F.Fab)
+      (effects (font (size 1 1) (thickness 0.15)))
+    )
+    (fp_text user %R (at 0 6.35 90) (layer F.Fab)
+      (effects (font (size 1 1) (thickness 0.15)))
+    )
+    (fp_line (start -1.8 14.45) (end -1.8 -1.8) (layer F.CrtYd) (width 0.05))
+    (fp_line (start 1.75 14.45) (end -1.8 14.45) (layer F.CrtYd) (width 0.05))
+    (fp_line (start 1.75 -1.8) (end 1.75 14.45) (layer F.CrtYd) (width 0.05))
+    (fp_line (start -1.8 -1.8) (end 1.75 -1.8) (layer F.CrtYd) (width 0.05))
+    (fp_line (start 0 -1.33) (end 1.33 -1.33) (layer F.SilkS) (width 0.12))
+    (fp_line (start 1.33 -1.33) (end 1.33 0) (layer F.SilkS) (width 0.12))
+    (fp_line (start 1.33 1.27) (end 1.33 14.03) (layer F.SilkS) (width 0.12))
+    (fp_line (start -1.33 14.03) (end 1.33 14.03) (layer F.SilkS) (width 0.12))
+    (fp_line (start -1.33 1.27) (end -1.33 14.03) (layer F.SilkS) (width 0.12))
+    (fp_line (start -1.33 1.27) (end 1.33 1.27) (layer F.SilkS) (width 0.12))
+    (fp_line (start -1.27 13.97) (end -1.27 -1.27) (layer F.Fab) (width 0.1))
+    (fp_line (start 1.27 13.97) (end -1.27 13.97) (layer F.Fab) (width 0.1))
+    (fp_line (start 1.27 -0.635) (end 1.27 13.97) (layer F.Fab) (width 0.1))
+    (fp_line (start 0.635 -1.27) (end 1.27 -0.635) (layer F.Fab) (width 0.1))
+    (fp_line (start -1.27 -1.27) (end 0.635 -1.27) (layer F.Fab) (width 0.1))
+    (pad 6 thru_hole oval (at 0 12.7) (size 1.7 1.7) (drill 1) (layers *.Cu *.Mask)
+      (net 1 "Net-(J1-Pad11)"))
+    (pad 5 thru_hole oval (at 0 10.16) (size 1.7 1.7) (drill 1) (layers *.Cu *.Mask)
+      (net 2 "Net-(J1-Pad10)"))
+    (pad 4 thru_hole oval (at 0 7.62) (size 1.7 1.7) (drill 1) (layers *.Cu *.Mask)
+      (net 5 "Net-(J1-Pad7)"))
+    (pad 3 thru_hole oval (at 0 5.08) (size 1.7 1.7) (drill 1) (layers *.Cu *.Mask)
+      (net 6 "Net-(J1-Pad5)"))
+    (pad 2 thru_hole oval (at 0 2.54) (size 1.7 1.7) (drill 1) (layers *.Cu *.Mask)
+      (net 3 "Net-(J1-Pad3)"))
+    (pad 1 thru_hole rect (at 0 0) (size 1.7 1.7) (drill 1) (layers *.Cu *.Mask)
+      (net 4 "Net-(J1-Pad1)"))
+    (model ${KISYS3DMOD}/Connector_PinSocket_2.54mm.3dshapes/PinSocket_1x06_P2.54mm_Vertical.wrl
+      (at (xyz 0 0 0))
+      (scale (xyz 1 1 1))
+      (rotate (xyz 0 0 0))
+    )
   )
   (module Connector_PinSocket_2.54mm:PinSocket_2x06_P2.54mm_Vertical (layer F.Cu)
@@
     )
   )
-  (gr_arc (start 25.4 36.83) (end 22.86 36.83) (angle -180) (layer Edge.Cuts) (width 0.1))
-  (gr_arc (start 25.4 16.51) (end 27.94 16.51) (angle -180) (layer Edge.Cuts) (width 0.1))
-  (gr_line (start 27.94 16.51) (end 27.94 36.83) (layer Edge.Cuts) (width 0.1))
+  (gr_arc (start 27.94 36.83) (end 27.94 39.37) (angle -90) (layer Edge.Cuts) (width 0.1))
+  (gr_line (start 25.4 39.37) (end 27.94 39.37) (layer Edge.Cuts) (width 0.1))
+  (gr_line (start 25.4 13.97) (end 27.94 13.97) (layer Edge.Cuts) (width 0.1))
+  (gr_arc (start 27.94 16.51) (end 30.48 16.51) (angle -90) (layer Edge.Cuts) (width 0.1))
+  (gr_arc (start 25.4 36.83) (end 22.86 36.83) (angle -90) (layer Edge.Cuts) (width 0.1))
+  (gr_arc (start 25.4 16.51) (end 25.4 13.97) (angle -90) (layer Edge.Cuts) (width 0.1))
+  (gr_line (start 30.48 16.51) (end 30.48 36.83) (layer Edge.Cuts) (width 0.1))
   (gr_line (start 22.86 36.83) (end 22.86 16.51) (layer Edge.Cuts) (width 0.1))
   (segment (start 26.67 33.02) (end 24.13 33.02) (width 1) (layer F.Cu) (net 1))
+  (segment (start 26.67 33.02) (end 29.21 33.02) (width 1) (layer F.Cu) (net 1))
   (segment (start 26.67 30.48) (end 24.13 30.48) (width 1) (layer F.Cu) (net 2))
+  (segment (start 26.67 30.48) (end 29.21 30.48) (width 1) (layer F.Cu) (net 2))
   (segment (start 26.67 22.86) (end 24.13 22.86) (width 1) (layer F.Cu) (net 3))
+  (segment (start 26.67 22.86) (end 29.21 22.86) (width 1) (layer F.Cu) (net 3))
   (segment (start 26.67 20.32) (end 24.13 20.32) (width 1) (layer F.Cu) (net 4))
+  (segment (start 26.67 20.32) (end 29.21 20.32) (width 1) (layer F.Cu) (net 4))
   (segment (start 26.67 27.94) (end 24.13 27.94) (width 1) (layer F.Cu) (net 5))
+  (segment (start 26.67 27.94) (end 29.21 27.94) (width 1) (layer F.Cu) (net 5))
   (segment (start 26.67 25.4) (end 24.13 25.4) (width 1) (layer F.Cu) (net 6))
+  (segment (start 26.67 25.4) (end 29.21 25.4) (width 1) (layer F.Cu) (net 6))
 )
