File: Hardware/SwitchboardConnector/SwitchboardConnector.sch (KiCad schematic (older format))
At the start: 1 part, among them J1 Conn_02x06_Odd_Even

Commit message: Further updates
Parts:
- added J2: Conn_01x06_Female, Connector_PinSocket_2.54mm:PinSocket_1x06_P2.54mm_Vertical, symbol Connector:Conn_01x06_Female
Connections:
- net at J1.1 (Pin_1), J1.2 (Pin_2): now also J2.1 (Pin_1)
- net at J1.10 (Pin_10), J1.9 (Pin_9): now also J2.5 (Pin_5)
- net at J1.11 (Pin_11), J1.12 (Pin_12): now also J2.6 (Pin_6)
- net at J1.3 (Pin_3), J1.4 (Pin_4): now also J2.2 (Pin_2)
- net at J1.5 (Pin_5), J1.6 (Pin_6): now also J2.3 (Pin_3)
- net at J1.7 (Pin_7), J1.8 (Pin_8): now also J2.4 (Pin_4)
Changed lines of the file:
@@
 	1    0    0    -1
 $EndComp
+$Comp
+L Connector:Conn_01x06_Female J2
+U 1 1 5E08914C
+P 2300 1200
+F 0 "J2" H 2328 1176 50  0000 L CNN
+F 1 "Conn_01x06_Female" H 2328 1085 50  0000 L CNN
+F 2 "Connector_PinSocket_2.54mm:PinSocket_1x06_P2.54mm_Vertical" H 2300 1200 50  0001 C CNN
+F 3 "~" H 2300 1200 50  0001 C CNN
+	1    2300 1200
+	1    0    0    -1
+$EndComp
+Wire Wire Line
+	1750 1000 2100 1000
+Connection ~ 1750 1000
+Wire Wire Line
+	1850 1100 2100 1100
+Connection ~ 1850 1100
+Wire Wire Line
+	1950 1200 2100 1200
+Connection ~ 1950 1200
+Wire Wire Line
+	1950 1300 2100 1300
+Connection ~ 1950 1300
+Wire Wire Line
+	1850 1400 2100 1400
+Connection ~ 1850 1400
+Wire Wire Line
+	1750 1500 2100 1500
+Connection ~ 1750 1500
 $EndSCHEMATC
